Commit message: work done: pointcloud stabilization (fail)

File: rotors_description/urdf/vi_sensor_base.xacro (robot description, xacro)
@@ -1,5 +1,5 @@
 <?xml version="1.0"?>
 <robot name="vi_sensor" xmlns:xacro="http://ros.org/wiki/xacro">
-  <xacro:property name="namespace" value="vi_sensor" />
+<!--  <xacro:property name="namespace" value="vi_sensor" />
   <xacro:include filename="$(find rotors_description)/urdf/component_snippets.xacro" />
   <link name="base_link">
@@ -11,5 +11,5 @@
     </collision>
     <visual>
-      <origin xyz="0 0 0" rpy="0 0 0" />
+      <origin xyz="0 0 0" rpy="0 0 0" />c
       <geometry>
         <box size="0.1 0.1 1.0" />
@@ -24,10 +24,10 @@
   </link>
   <xacro:vi_sensor_macro
-    namespace="${namespace}"
-    parent_link="base_link"
+    namespace="${namespace}/base_link"
+    parent_link="${namespace}/gimbal_base_link"
     enable_cameras="$(arg enable_cameras)"
     enable_depth="$(arg enable_depth)"
     enable_ground_truth="$(arg enable_ground_truth)">
-    <origin xyz="0.0 0.0 0.8" rpy="0 0 0" />
-  </xacro:vi_sensor_macro>
+    <origin xyz="0.0 0.0 -0.030" rpy="0.0 1.570796 0.0" />
+  </xacro:vi_sensor_macro> -->
 </robot>
