Commit message: using tf transformer for stabilized pointcloud2

File: rotors_description/urdf/multirotor_base.xacro (robot description, xacro)
@@ -54,5 +54,5 @@
       <child link="${robot_namespace}/gimbal_base_link" />
       <origin xyz="0 0 0" rpy="0 0 0" />
-      <axis xyz="0 1 0" />
+      <axis xyz="0 1.570796 0" />
     </joint>
     <gazebo>
