Commit message: fix: some fk/ik related issue

File: rotors_description/urdf/firefly_large_landing_gear.xacro (robot description, xacro)
@@ -185,5 +185,5 @@
     <inertial>
       <origin rpy="0.0 0.0 0.0" xyz="0.0 0.0 0.0"/>
-      <mass value="0.0001" />
+      <mass value="0.0230" />
       <inertia ixx="0.0021150000" iyy="0.0006921000" izz="0.0025240000" ixy="-0.0000163500" ixz="0.0000006998" iyz="0.0000464200" />
     </inertial>
@@ -229,5 +229,5 @@
     <inertial>
       <origin rpy="0.0 0.0 0.0" xyz="0.0 0.0 0.0"/>
-      <mass value="0.0001" />
+      <mass value="0.0230" />
       <inertia ixx="0.0021150000" iyy="0.0006921000" izz="0.0025240000" ixy="-0.0000163500" ixz="0.0000006998" iyz="0.0000464200" />
     </inertial>
@@ -245,5 +245,5 @@
     moment_constant="${moment_constant}"
     parent="${namespace}/base_link"
-    mass_rotor="${mass_rotor}"
+    mass_rotor="${mass_rotor+0.0025}"
     radius_rotor="${radius_rotor}"
     time_constant_up="${time_constant_up}"

File: rotors_description/urdf/mav_with_vi_sensor_robot_arm_srdf.xacro (robot description, xacro)
@@ -2,4 +2,5 @@
   <xacro:macro name="wx250s_arm">
     <group name="wx250s_arm">
+      <joint name="virtual_joint"/>
       <joint name="wx250s_waist" />
       <joint name="wx250s_shoulder"/>
@@ -9,5 +10,4 @@
       <joint name="wx250s_wrist_rotate"/>
     </group>
-    <virtual_joint name="virtual_joint" type="floating" parent_frame="world" child_link="firefly/base_link" />
     <group_state name="home" group="wx250s_arm">
       <joint name="wx250s_waist" value="0.0" />

File: rotors_description/urdf/mav_with_vi_sensor_robot_arm_urdf.xacro (robot description, xacro)
@@ -34,5 +34,5 @@
     <link name="firefly/base_link"/>
     <!-- making the base joint for the manipulator  -->
-    <joint name="fixed" type="fixed">
+    <joint name="virtual_joint" type="fixed">
       <parent link="firefly/base_link"/>
       <child link="firefly/wx250s/base_link"/>
