Commit message: work done: vi sensor check and manual contorl check

File: rotors_description/urdf/component_snippets.xacro (robot description, xacro)
@@ -563,5 +563,5 @@
       image_width="752"
       image_height="480"
-      image_format="L8"
+      image_format="B8G8R8"
       min_distance="0.02"
       max_distance="30"
@@ -584,5 +584,5 @@
       image_width="752"
       image_height="480"
-      image_format="L8"
+      image_format="B8G8R8"
       min_distance="0.02"
       max_distance="${max_range}"

File: rotors_description/urdf/vi_sensor_base.xacro (robot description, xacro)
@@ -29,5 +29,5 @@
     enable_depth="$(arg enable_depth)"
     enable_ground_truth="$(arg enable_ground_truth)">
-    <origin xyz="0.0 0.0 0.6" rpy="0 0 0" />
+    <origin xyz="0.0 0.0 0.8" rpy="0 0 0" />
   </xacro:vi_sensor_macro>
 </robot>

Commit message: work done: gimbal_base_link and plugin, just compiled

File: rotors_description/urdf/component_snippets.xacro (robot description, xacro)
@@ -18,4 +18,23 @@
 <robot xmlns:xacro="http://ros.org/wiki/xacro">
   <xacro:property name="pi" value="3.14159265359" />
+  <!-- Macro to add gimbal base link -->
+  <!-- <xacro:macro name="gimbal_macro" params="namespace *origin">
+    <link name="${namespace}/gimbal_base_link">
+      <inertial>
+        <mass value="0.1" />
+        <inertia ixx="1e-4" ixy="0.0" ixz="0.0" iyy="1e-4" iyz="0.0" izz="1e-4" />
+      </inertial>
+    </link>
+    <joint name="${namespace}/gimbal_pitch_joint" type="continuous">
+      <parent link="${namespace}/base_link" />
+      <child link="${namespace}/gimbal_base_link" />
+      <origin xyz="0 0 0" rpy="0 0 0" />
+      <axis xyz="0 1 0" />
+    </joint>
+    <gazebo>
+      <plugin name="gimbal_controller" filename="libgimbal_plugin.so">
+      </plugin>
+    </gazebo>
+  </xacro:macro>-->
   <!-- Macro to add logging to a bag file. -->
   <xacro:macro name="bag_plugin_macro"

File: rotors_description/urdf/firefly.xacro (robot description, xacro)
@@ -48,4 +48,8 @@
   <!-- Included URDF Files -->
   <xacro:include filename="$(find rotors_description)/urdf/multirotor_base.xacro" />
+  <!-- Included gimbal base link -->
+  <!--<xacro:gimbal_macro namespace="${namespace}">
+    <origin xyz="0 0 -0.5" rpy="0 0 0" />
+  </xacro:gimbal_macro> -->
   <!-- Instantiate multirotor_base_macro once -->
   <xacro:multirotor_base_macro

Commit message: work done: add gimbal base

File: rotors_description/urdf/component_snippets.xacro (robot description, xacro)
@@ -18,23 +18,4 @@
 <robot xmlns:xacro="http://ros.org/wiki/xacro">
   <xacro:property name="pi" value="3.14159265359" />
-  <!-- Macro to add gimbal base link -->
-  <!-- <xacro:macro name="gimbal_macro" params="namespace *origin">
-    <link name="${namespace}/gimbal_base_link">
-      <inertial>
-        <mass value="0.1" />
-        <inertia ixx="1e-4" ixy="0.0" ixz="0.0" iyy="1e-4" iyz="0.0" izz="1e-4" />
-      </inertial>
-    </link>
-    <joint name="${namespace}/gimbal_pitch_joint" type="continuous">
-      <parent link="${namespace}/base_link" />
-      <child link="${namespace}/gimbal_base_link" />
-      <origin xyz="0 0 0" rpy="0 0 0" />
-      <axis xyz="0 1 0" />
-    </joint>
-    <gazebo>
-      <plugin name="gimbal_controller" filename="libgimbal_plugin.so">
-      </plugin>
-    </gazebo>
-  </xacro:macro>-->
   <!-- Macro to add logging to a bag file. -->
   <xacro:macro name="bag_plugin_macro"

File: rotors_description/urdf/firefly.xacro (robot description, xacro)
@@ -48,8 +48,4 @@
   <!-- Included URDF Files -->
   <xacro:include filename="$(find rotors_description)/urdf/multirotor_base.xacro" />
-  <!-- Included gimbal base link -->
-  <!--<xacro:gimbal_macro namespace="${namespace}">
-    <origin xyz="0 0 -0.5" rpy="0 0 0" />
-  </xacro:gimbal_macro> -->
   <!-- Instantiate multirotor_base_macro once -->
   <xacro:multirotor_base_macro

File: rotors_description/urdf/multirotor_base.xacro (robot description, xacro)
@@ -35,4 +35,31 @@
     params="robot_namespace mass body_width body_height use_mesh_file mesh_file *inertia">
     <link name="${robot_namespace}/base_link"></link>
+    <!-- Included gimbal base link -->
+    <link name="${robot_namespace}/gimbal_base_link">
+      <inertial>
+        <origin xyz="0 0 -0.025" rpy="0 0 0" />
+        <mass value="0.1" />
+        <inertia ixx="5e-2" ixy="0.0" ixz="0.0" iyy="5e-2" iyz="0.0" izz="5e-2" />
+      </inertial>
+      <visual>
+        <origin xyz="0 0 -0.025" rpy="0 0 0"/>
+        <geometry>
+          <cylinder radius="0.025" length="0.01"/>
+        </geometry>
+        <material name="white"/>
+      </visual>
+    </link>
+    <joint name="${robot_namespace}/gimbal_pitch_joint" type="continuous">
+      <parent link="${robot_namespace}/base_link" />
+      <child link="${robot_namespace}/gimbal_base_link" />
+      <origin xyz="0 0 0" rpy="0 0 0" />
+      <axis xyz="0 1 0" />
+    </joint>
+    <gazebo>
+      <plugin name="gimbal_controller_plugin" filename="librotors_gazebo_gimbal_plugin.so">
+        <linkBaseName>${robot_namespace}/base_link</linkBaseName>
+        <linkPitchName>${robot_namespace}/gimbal_base_link</linkPitchName>
+      </plugin>
+    </gazebo>
     <joint name="${robot_namespace}/base_joint" type="fixed">
       <origin xyz="0 0 0" rpy="0 0 0" />

Commit message: working: adding leddar vu8

File: rotors_description/urdf/component_snippets.xacro (robot description, xacro)
@@ -32,4 +32,62 @@
     </gazebo>
   </xacro:macro>
+  <!-- leddar vu8 8-segment sensor -->
+<!--   <xacro:macro name="lidar_leddar_vu8_macro" params="namespace parent_link lidar_name lidar_topic min_angle max_angle min_range max_range *origin">
+    <link name="${lidar_name}/lidar_link">
+      <visual name="visual">
+        <origin xyz="0 0 0" rpy="${pi/2} 0 0" />
+        <geometry>
+          <mesh filename="package://rotors_description/meshes/leddarvu.dae" scale="1 1 1" />
+        </geometry>
+      </visual>
+    </link>
+    <joint name="${lidar_name}/lidar_joint" type="fixed">
+      <xacro:insert_block name="origin" />
+      <parent link="${parent_link}" />
+      <child link="${lidar_name}/lidar_link" />
+    </joint>
+    <link name="${lidar_name}/lidar_optical_link">
+    </link>
+    <joint name="${lidar_name}/lidar_optical_joint" type="fixed">
+      <origin xyz="0 0 0" rpy="0 0 0" />
+      <parent link="${lidar_name}/lidar_link" />
+      <child link="${lidar_name}/lidar_optical_link" />
+    </joint>
+    <gazebo reference="${lidar_name}/lidar_optical_link">
+      <sensor type="ray" name="${lidar_name}_lidar">
+        <pose>0 0 0 0 0 0</pose>
+        <visualize>true</visualize>
+        <update_rate>100</update_rate>
+        <ray>
+          <scan>
+            <horizontal>
+              <samples>8</samples>
+              <resolution>30</resolution>
+              <min_angle>${min_angle}</min_angle>
+              <max_angle>${max_angle}</max_angle>
+            </horizontal>
+          </scan>
+          <range>
+            <min>0.1</min>
+            <max>${max_range + 1}</max>
+            <resolution>0.01</resolution>
+          </range>
+          <noise>
+            <type>gaussian</type>
+            <mean>0.0</mean>
+            <stddev>0.01</stddev>
+          </noise>
+        </ray>
+        <plugin name="gazebo_leddar_vu8_lidar_plugin" filename="libgazebo_leddar_vu8_lidar_plugin.so">
+          <lidar_topic>${lidar_topic}</lidar_topic>
+          <min_range>${min_range}</min_range>
+          <max_range>${max_range}</max_range>
+          <min_angle>${min_angle}</min_angle>
+          <max_angle>${max_angle}</max_angle>
+        </plugin>
+        <always_on>1</always_on>
+      </sensor>
+    </gazebo>
+  </xacro:macro>   -->
   <!-- Macro to add a camera. -->
   <xacro:macro name="camera_macro"

Commit message: work done: joystick control within lee_position_controller, temporary

File: rotors_description/urdf/component_snippets.xacro (robot description, xacro)
@@ -33,9 +33,10 @@
   </xacro:macro>
   <!-- leddar vu8 8-segment sensor -->
-<!--   <xacro:macro name="lidar_leddar_vu8_macro" params="namespace parent_link lidar_name lidar_topic min_angle max_angle min_range max_range *origin">
+  <xacro:macro name="lidar_leddar_vu8_macro" params="namespace parent_link lidar_name lidar_topic min_angle max_angle min_range max_range *origin">
     <link name="${lidar_name}/lidar_link">
       <visual name="visual">
         <origin xyz="0 0 0" rpy="${pi/2} 0 0" />
         <geometry>
+          <!-- <cylinder radius="0.005" length="0.005"/>  -->
           <mesh filename="package://rotors_description/meshes/leddarvu.dae" scale="1 1 1" />
         </geometry>
@@ -89,5 +90,5 @@
       </sensor>
     </gazebo>
-  </xacro:macro>   -->
+  </xacro:macro>
   <!-- Macro to add a camera. -->
   <xacro:macro name="camera_macro"
@@ -687,4 +688,5 @@
       <sensor type="depth" name="${namespace}_camera_{camera_suffix}">
         <always_on>true</always_on>
+        <visualize>true</visualize>
         <update_rate>${frame_rate}</update_rate>
         <camera>

Commit message: working: adding manipulator

File: rotors_description/urdf/component_snippets.xacro (robot description, xacro)
@@ -28,7 +28,140 @@
         <frameId>${namespace}/base_link</frameId>
         <rotorVelocitySlowdownSim>${rotor_velocity_slowdown_sim}</rotorVelocitySlowdownSim>
-	<waitToRecordBag>${wait_to_record_bag}</waitToRecordBag>
+	      <waitToRecordBag>${wait_to_record_bag}</waitToRecordBag>
       </plugin>
     </gazebo>
+  </xacro:macro>
+  <!-- Macro to add wx250s robot arm. -->
+  <xacro:macro name="wx250s_robot_arm" params="namespace parent_link x_offset z_offset">
+    <xacro:arg name="use_default_gripper_bar" default="true"/>
+    <xacro:arg name="use_default_gripper_fingers" default="true"/>
+    <joint name="fixed" type="fixed">
+      <parent link="${parent_link}"/>
+      <child link="${namespace}/wx250s/base_link"/>
+    </joint>
+    <link name="${namespace}/wx250s/base_link">
+      <visual>
+        <origin rpy="${pi} 0 ${-pi/2}" xyz="${x_offset} 0.0 ${z_offset}"/>
+        <geometry>
+          <mesh filename="package://rotors_description/meshes/wx250s/WXSA-250-M-1-Base.stl" scale="0.001 0.001 0.001"/>
+        </geometry>
+      </visual>
+      <collision>
+        <origin rpy="${pi} 0 ${-pi/2}" xyz="${x_offset} 0.0 ${z_offset}"/>
+        <geometry>
+          <mesh filename="package://rotors_description/meshes/wx250s/WXSA-250-M-1-Base.stl" scale="0.001 0.001 0.001"/>
+        </geometry>
+      </collision>
+      <inertial>
+        <origin rpy="${pi} 0 ${-pi/2}" xyz="0.0 0.0 0.0"/>
+        <mass value="0.001" />
+        <inertia ixx="0.0021150000" iyy="0.0006921000" izz="0.0025240000" ixy="-0.0000163500" ixz="0.0000006998" iyz="0.0000464200" />
+      </inertial>
+    </link>
+    <joint name="wx250s_waist" type="revolute">
+      <axis xyz="0 0 1"/>
+      <limit effort="100" lower="${-pi}" upper="${pi}" velocity="${pi}"/>
+      <origin rpy="${pi} 0 ${-pi/2}" xyz="${x_offset} 0.0 ${z_offset+0.0716}"/>
+      <parent link="${namespace}/wx250s/base_link"/>
+      <child link="${namespace}/wx250s/shoulder_link"/>
+    </joint>
+    <transmission name="wx250s_trans_waist">
+      <type>transmission_interface/SimpleTransmission</type>
+      <joint name="wx250s_waist">
+        <hardwareInterface>hardware_interface/EffortJointInterface</hardwareInterface>
+      </joint>
+      <actuator name="wx250s_waist_motor">
+        <mechanicalReduction>1</mechanicalReduction>
+      </actuator>
+    </transmission>
+    <link name="${namespace}/wx250s/shoulder_link">
+      <visual>
+        <origin rpy="0.0 0.0 0.0" xyz="0 0 0.137"/>
+        <geometry>
+          <mesh filename="package://rotors_description/meshes/wx250s/WXSA-250-M-2-Shoulder.stl" scale="0.001 0.001 0.001"/>
+        </geometry>
+      </visual>
+      <collision>
+        <origin rpy="0.0 0.0 0.0" xyz="0 0 0.137"/>
+        <geometry>
+          <mesh filename="package://rotors_description/meshes/wx250s/WXSA-250-M-2-Shoulder.stl" scale="0.001 0.001 0.001"/>
+        </geometry>
+      </collision>
+      <inertial>
+        <origin rpy="0.0 0.0 0.0" xyz="0 0 0.0"/>
+        <mass value="0.001" />
+        <inertia ixx="0.0003790000" iyy="0.0005557000" izz="0.0005889000" ixy="0.0000000022" ixz="-0.0000003561" iyz="0.0000012245" />
+      </inertial>
+    </link>
+    <joint name="wx250s_shoulder" type="revolute">
+      <axis xyz="1 0 0"/>
+      <limit effort="100" lower="${radians(-108)}" upper="${radians(114)}" velocity="${pi}"/>
+      <origin rpy="0 0 0" xyz="0 0 0.165"/>
+      <parent link="${namespace}/wx250s/shoulder_link"/>
+      <child link="${namespace}/wx250s/upper_arm_link"/>
+    </joint>
+    <transmission name="wx250s_trans_shoulder">
+      <type>transmission_interface/SimpleTransmission</type>
+      <joint name="wx250s_shoulder">
+        <hardwareInterface>hardware_interface/EffortJointInterface</hardwareInterface>
+      </joint>
+      <actuator name="wx250s_shoulder_motor">
+        <mechanicalReduction>1</mechanicalReduction>
+      </actuator>
+    </transmission>
+    <link name="${namespace}/wx250s/upper_arm_link">
+      <visual>
+        <origin rpy="0.0 0.0 0.0" xyz="0.0 0.0 0.0"/>
+        <geometry>
+          <mesh filename="package://rotors_description/meshes//wx250s/WXSA-250-M-3-UA.stl" scale="0.001 0.001 0.001"/>
+        </geometry>
+      </visual>
+      <collision>
+        <origin rpy="0.0 0.0 0.0" xyz="0.0 0.0 0.0"/>
+        <geometry>
+          <mesh filename="package://rotors_description/meshes//wx250s/WXSA-250-M-3-UA.stl" scale="0.001 0.001 0.001"/>
+        </geometry>
+      </collision>
+      <inertial>
+        <origin rpy="0.0 0.0 0.0" xyz="0.0 0.0 0.0"/>
+        <mass value="0.001" />
+        <inertia ixx="0.0034630000" iyy="0.0035870000" izz="0.0004566000" ixy="-0.0000000001" ixz="-0.0000000002" iyz="0.0004272000" />
+      </inertial>
+    </link>
+   <joint name="wx250s_elbow" type="revolute">
+      <axis xyz="0 0 1"/>
+      <limit effort="100" lower="${radians(-92)}" upper="${radians(123)}" velocity="${pi}"/>
+      <origin rpy="0 ${pi/2} 0" xyz="0.0 -0.05 0.25"/>
+      <parent link="${namespace}/wx250s/upper_arm_link"/>
+      <child link="${namespace}/wx250s/upper_forearm_link"/>
+    </joint>
+    <transmission name="wx250s_trans_elbow">
+      <type>transmission_interface/SimpleTransmission</type>
+      <joint name="wx250s_elbow">
+        <hardwareInterface>hardware_interface/EffortJointInterface</hardwareInterface>
+      </joint>
+      <actuator name="wx250s_elbow_motor">
+        <mechanicalReduction>1</mechanicalReduction>
+      </actuator>
+    </transmission>
+    <link name="${namespace}/wx250s/upper_forearm_link">
+      <visual>
+        <origin rpy="${pi/2} ${pi} ${pi/2}" xyz="0.0 0.0 0.0"/>
+        <geometry>
+          <mesh filename="package://rotors_description/meshes/wx250s/WXSA-250-M-4-UF.stl" scale="0.001 0.001 0.001"/>
+        </geometry>
+      </visual>
+      <collision>
+        <origin rpy="${pi/2} ${pi} ${pi/2}" xyz="0.0 0.0 0.0"/>
+        <geometry>
+          <mesh filename="package://rotors_description/meshes/wx250s/WXSA-250-M-4-UF.stl" scale="0.001 0.001 0.001"/>
+        </geometry>
+      </collision>
+      <inertial>
+        <origin rpy="0.0 0.0 0.0" xyz="0.0 0.0 0.0"/>
+        <mass value="0.001" />
+        <inertia ixx="0.0000397100" iyy="0.0008878000" izz="0.0008880000" ixy="0.0000023528" ixz="0" iyz="0" />
+      </inertial>
+    </link>
   </xacro:macro>
   <!-- leddar vu8 8-segment sensor -->
