Commit message: work done: aerial manipulator version v1.0

File: rotors_description/urdf/component_snippets.xacro (robot description, xacro)
@@ -32,12 +32,13 @@
     </gazebo>
   </xacro:macro>
+  <!--///////////////////////////////////////////////////////////////////////////////////////////////////////////////////////////////// -->
   <!-- Macro to add wx250s robot arm. -->
   <xacro:macro name="wx250s_robot_arm" params="namespace parent_link x_offset z_offset">
-    <xacro:arg name="use_default_gripper_bar" default="true"/>
-    <xacro:arg name="use_default_gripper_fingers" default="true"/>
+    <!-- making the base joint for the manipulator  -->
     <joint name="fixed" type="fixed">
       <parent link="${parent_link}"/>
       <child link="${namespace}/wx250s/base_link"/>
     </joint>
+    <!-- making the base link for the manipulator, lower deck  -->
     <link name="${namespace}/wx250s/base_link">
       <visual>
@@ -59,4 +60,5 @@
       </inertial>
     </link>
+    <!-- making the waist joint -->
     <joint name="wx250s_waist" type="revolute">
       <axis xyz="0 0 1"/>
@@ -66,4 +68,5 @@
       <child link="${namespace}/wx250s/shoulder_link"/>
     </joint>
+    <!-- making the waist servo -->
     <transmission name="wx250s_trans_waist">
       <type>transmission_interface/SimpleTransmission</type>
@@ -75,4 +78,5 @@
       </actuator>
     </transmission>
+    <!-- making the shoulder link -->
     <link name="${namespace}/wx250s/shoulder_link">
       <visual>
@@ -94,4 +98,5 @@
       </inertial>
     </link>
+    <!-- making the shoulder joint -->
     <joint name="wx250s_shoulder" type="revolute">
       <axis xyz="1 0 0"/>
@@ -101,4 +106,5 @@
       <child link="${namespace}/wx250s/upper_arm_link"/>
     </joint>
+    <!-- making the shoulder servo -->
     <transmission name="wx250s_trans_shoulder">
       <type>transmission_interface/SimpleTransmission</type>
@@ -110,4 +116,5 @@
       </actuator>
     </transmission>
+    <!-- making the upper arm link, between the shoulder and the elbow -->
     <link name="${namespace}/wx250s/upper_arm_link">
       <visual>
@@ -129,5 +136,6 @@
       </inertial>
     </link>
-   <joint name="wx250s_elbow" type="revolute">
+    <!-- making the elbow joint, between the shoulder and the elbow -->
+    <joint name="wx250s_elbow" type="revolute">
       <axis xyz="0 0 1"/>
       <limit effort="100" lower="${radians(-92)}" upper="${radians(123)}" velocity="${pi}"/>
@@ -136,4 +144,5 @@
       <child link="${namespace}/wx250s/upper_forearm_link"/>
     </joint>
+    <!-- making the elbow servo, between the shoulder and the elbow -->
     <transmission name="wx250s_trans_elbow">
       <type>transmission_interface/SimpleTransmission</type>
@@ -145,4 +154,5 @@
       </actuator>
     </transmission>
+    <!-- making the upper forearm link, for the rotation of the elbow -->
     <link name="${namespace}/wx250s/upper_forearm_link">
       <visual>
@@ -164,5 +174,240 @@
       </inertial>
     </link>
-  </xacro:macro>
+    <!-- making the forearm roll joint, for the rotation of the elbow -->
+    <joint name="wx250s_forearm_roll" type="revolute">
+      <axis xyz="0 -1 0"/>
+      <limit effort="100" lower="${radians(-180)}" upper="${radians(180)}" velocity="${pi}"/>
+      <origin rpy="0 0 0" xyz="0.0 -0.175 0.0"/>
+      <parent link="${namespace}/wx250s/upper_forearm_link"/>
+      <child link="${namespace}/wx250s/lower_forearm_link"/>
+    </joint>
+    <!-- making the forearm roll servo, for the rotation of the elbow -->
+    <transmission name="wx250s_trans_forearm_roll">
+      <type>transmission_interface/SimpleTransmission</type>
+      <joint name="wx250s_forearm_roll">
+        <hardwareInterface>hardware_interface/EffortJointInterface</hardwareInterface>
+      </joint>
+      <actuator name="wx250s_forearm_roll_motor">
+        <mechanicalReduction>1</mechanicalReduction>
+      </actuator>
+    </transmission>
+    <!-- making the lower forearm link, for the rotation of the wrist -->
+    <link name="${namespace}/wx250s/lower_forearm_link">
+      <visual>
+        <origin rpy="${-pi/2} ${-pi} ${pi/2}" xyz="0 0 0"/>
+        <geometry>
+          <mesh filename="package://rotors_description/meshes/wx250s/WXSA-250-M-5-LF.stl" scale="0.001 0.001 0.001"/>
+        </geometry>
+      </visual>
+      <collision>
+        <origin rpy="${-pi/2} ${-pi} ${pi/2}" xyz="0 0 0"/>
+        <geometry>
+          <mesh filename="package://rotors_description/meshes/wx250s/WXSA-250-M-5-LF.stl" scale="0.001 0.001 0.001"/>
+        </geometry>
+      </collision>
+      <inertial>
+        <origin rpy="0 0 0" xyz="0.0 0.0 0"/>
+        <mass value="0.001" />
+        <inertia ixx="0.0000636900" iyy="0.0001677000" izz="0.0001834000" ixy="-0.0000229200" ixz="0" iyz="0" />
+      </inertial>
+    </link>
+    <!-- making the wrist joint, for the rotation of the wrist -->
+    <joint name="wx250s_wrist_angle" type="revolute">
+      <axis xyz="-1 0 0"/>
+      <limit effort="100" lower="${radians(-123)}" upper="${radians(100)}" velocity="${pi}"/>
+      <origin rpy="0.0 ${pi/2} 0.0" xyz="0.0 -0.075 0.0"/>
+      <parent link="${namespace}/wx250s/lower_forearm_link"/>
+      <child link="${namespace}/wx250s/wrist_link"/>
+    </joint>
+    <!-- making the wrist servo, for the rotation of the wrist -->
+    <transmission name="wx250s_trans_wrist_angle">
+      <type>transmission_interface/SimpleTransmission</type>
+      <joint name="wx250s_wrist_angle">
+        <hardwareInterface>hardware_interface/EffortJointInterface</hardwareInterface>
+      </joint>
+      <actuator name="wx250s_wrist_angle_motor">
+        <mechanicalReduction>1</mechanicalReduction>
+      </actuator>
+    </transmission>
+    <!-- making the wrist link, for the rotation of the wrist -->
+    <link name="${namespace}/wx250s/wrist_link">
+      <visual>
+        <origin rpy="0 0 0" xyz="0 0 0"/>
+        <geometry>
+          <mesh filename="package://rotors_description/meshes/wx250s/WXSA-250-M-6-Wrist.stl" scale="0.001 0.001 0.001"/>
+        </geometry>
+        <material name="interbotix_black"/>
+      </visual>
+      <collision>
+        <origin rpy="0 0 0" xyz="0 0 0"/>
+        <geometry>
+          <mesh filename="package://rotors_description/meshes/wx250s/WXSA-250-M-6-Wrist.stl" scale="0.001 0.001 0.001"/>
+        </geometry>
+      </collision>
+      <inertial>
+        <origin rpy="0 0 0" xyz="0.0423600000 0.0000106630 -0.0105770000"/>
+        <mass value="0.001" />
+        <inertia ixx="0.0000308200" iyy="0.0000282200" izz="0.0000315200" ixy="0.0000000191" ixz="0.0000000023" iyz="0.0000025481" />
+      </inertial>
+    </link>
+    <!-- making the wrist joint, for the rotation of the wrist -->
+    <joint name="wx250s_wrist_rotate" type="revolute">
+      <axis xyz="0 1 0"/>
+      <limit effort="100" lower="${-pi}" upper="${pi}" velocity="${pi}"/>
+      <origin rpy="0 0 0" xyz="0.0 0.0 0.0"/>
+      <parent link="${namespace}/wx250s/wrist_link"/>
+      <child link="${namespace}/wx250s/gripper_link"/>
+    </joint>
+    <!-- making the wrist servo, for the rotation of the wrist -->
+    <transmission name="wx250s_trans_wrist_rotate">
+      <type>transmission_interface/SimpleTransmission</type>
+      <joint name="wx250s_wrist_rotate">
+        <hardwareInterface>hardware_interface/EffortJointInterface</hardwareInterface>
+      </joint>
+      <actuator name="wx250s_wrist_rotate_motor">
+        <mechanicalReduction>1</mechanicalReduction>
+      </actuator>
+    </transmission>
+    <link name="${namespace}/wx250s/gripper_link">
+      <visual>
+        <origin rpy="0 0 0" xyz="0 -0.0448 0"/>
+        <geometry>
+          <mesh filename="package://rotors_description/meshes/wx250s/WXSA-250-M-7-Gripper.stl" scale="0.001 0.001 0.001"/>
+        </geometry>
+      </visual>
+      <collision>
+        <origin rpy="0 0 0" xyz="0 -0.0448 0"/>
+        <geometry>
+          <mesh filename="package://rotors_description/meshes/wx250s/WXSA-250-M-7-Gripper.stl" scale="0.001 0.001 0.001"/>
+        </geometry>
+      </collision>
+      <inertial>
+        <origin rpy="0 0 0" xyz="0.0216310000 0.0000002516 0.0114100000"/>
+        <mass value="0.001" />
+        <inertia ixx="0.0000253700" iyy="0.0000183600" izz="0.0000167400" ixy="0.0000000000" ixz="0.0000000000" iyz="0.0000004340" />
+      </inertial>
+    </link>
+    <joint name="wx250s_ee_arm" type="fixed">
+      <axis xyz="0 1 0"/>
+      <origin rpy="0 0 0" xyz="0 0 0"/>
+      <parent link="${namespace}/wx250s/gripper_link"/>
+      <child link="${namespace}/wx250s/ee_arm_link"/>
+    </joint>
+    <link name="${namespace}/wx250s/ee_arm_link">
+      <inertial>
+        <mass value="0.001" />
+        <inertia ixx="0.001" iyy="0.001" izz="0.001" ixy="0" ixz="0" iyz="0" />
+      </inertial>
+    </link>
+    <joint name="wx250s_gripper_bar" type="fixed">
+      <axis xyz="0 1 0"/>
+      <origin rpy="0 0 0" xyz="0 0 0"/>
+      <parent link="${namespace}/wx250s/ee_arm_link"/>
+      <child link="${namespace}/wx250s/gripper_bar_link"/>
+    </joint>
+    <link name="${namespace}/wx250s/gripper_bar_link">
+      <visual>
+        <origin rpy="0 0 0" xyz="0 -0.042 0"/>
+        <geometry>
+          <mesh filename="package://rotors_description/meshes/wx250s/WXSA-250-M-9-Gripper-Bar.stl" scale="0.001 0.001 0.001"/>
+        </geometry>
+      </visual>
+      <collision>
+        <origin rpy="0 0 0" xyz="0 -0.042 0"/>
+        <geometry>
+          <mesh filename="package://rotors_description/meshes/wx250s/WXSA-250-M-9-Gripper-Bar.stl" scale="0.001 0.001 0.001"/>
+        </geometry>
+      </collision>
+      <inertial>
+        <origin rpy="0 0 0" xyz="0.0096870000 0.0000008177 0.0049620000"/>
+        <mass value="0.001" />
+        <inertia ixx="0.0000074125" iyy="0.0000284300" izz="0.0000286000" ixy="-0.0000000008" ixz="-0.0000000006" iyz="-0.0000013889" />
+      </inertial>
+    </link>
+    <joint name="wx250s_ee_bar" type="fixed">
+      <axis xyz="0 1 0"/>
+      <origin rpy="0 0 0" xyz="0 0 0"/>
+      <parent link="${namespace}/wx250s/gripper_bar_link"/>
+      <child link="${namespace}/wx250s/fingers_link"/>
+    </joint>
+    <link name="${namespace}/wx250s/fingers_link">
+      <inertial>
+        <mass value="0.001" />
+        <inertia ixx="0.001" iyy="0.001" izz="0.001" ixy="0" ixz="0" iyz="0" />
+      </inertial>
+    </link>
+    <joint name="wx250s_left_finger" type="prismatic">
+      <axis xyz="1 0 0"/>
+      <limit effort="10" lower="-0.0" upper="0.1" velocity="0.1"/>
+      <origin rpy="0 0 0" xyz="0 0 0"/>
+      <parent link="${namespace}/wx250s/fingers_link"/>
+      <child link="${namespace}/wx250s/left_finger_link"/>
+    </joint>
+    <transmission name="wx250s_trans_left_finger">
+      <type>transmission_interface/SimpleTransmission</type>
+      <joint name="wx250s_left_finger">
+        <hardwareInterface>hardware_interface/EffortJointInterface</hardwareInterface>
+      </joint>
+      <actuator name="wx250s_left_finger_motor">
+        <mechanicalReduction>1</mechanicalReduction>
+      </actuator>
+    </transmission>
+    <link name="${namespace}/wx250s/left_finger_link">
+      <visual>
+        <origin rpy="0 ${pi} ${-pi/2}" xyz="-0.05 -0.12 0"/>
+        <geometry>
+          <mesh filename="package://rotors_description/meshes/wx250s/WXSA-250-M-10-Finger.stl" scale="0.001 0.001 0.001"/>
+        </geometry>
+        <material name="interbotix_black"/>
+      </visual>
+      <collision>
+        <origin rpy="0 ${pi} ${-pi/2}" xyz="-0.05 -0.12 0"/>
+        <geometry>
+          <mesh filename="package://rotors_description/meshes/wx250s/WXSA-250-M-10-Finger.stl" scale="0.001 0.001 0.001"/>
+        </geometry>
+      </collision>
+      <inertial>
+        <origin rpy="0 0 0" xyz="0.0138160000 0.0000000000 0.0000000000"/>
+          <mass value="0.016246" />
+        <inertia ixx="0.0000047310" iyy="0.0000015506" izz="0.0000037467" ixy="-0.0000004560" ixz="0.0000000000" iyz="0.0000000000" />
+      </inertial>
+    </link>
+    <joint name="wx250s_right_finger" type="prismatic">
+      <axis xyz="-1 0 0"/>
+      <limit effort="10" lower="-0.0" upper="0.1" velocity="0.1"/>
+      <origin rpy="0 0 0" xyz="0 0 0"/>
+      <parent link="${namespace}/wx250s/fingers_link"/>
+      <child link="${namespace}/wx250s/right_finger_link"/>
+    </joint>
+    <transmission name="wx250s_trans_right_finger">
+      <type>transmission_interface/SimpleTransmission</type>
+      <joint name="wx250s_right_finger">
+        <hardwareInterface>hardware_interface/EffortJointInterface</hardwareInterface>
+      </joint>
+      <actuator name="wx250s_right_finger_motor">
+        <mechanicalReduction>1</mechanicalReduction>
+      </actuator>
+    </transmission>
+    <link name="${namespace}/wx250s/right_finger_link">
+      <visual>
+        <origin rpy="${-pi} ${-pi} ${-pi/2}" xyz="0.05 -0.12 0"/>
+        <geometry>
+          <mesh filename="package://rotors_description/meshes/wx250s/WXSA-250-M-10-Finger.stl" scale="0.001 0.001 0.001"/>
+        </geometry>
+      </visual>
+      <collision>
+        <origin rpy="${-pi} ${-pi} ${-pi/2}" xyz="0.05 -0.12 0"/>
+        <geometry>
+          <mesh filename="package://rotors_description/meshes/wx250s/WXSA-250-M-10-Finger.stl" scale="0.001 0.001 0.001"/>
+        </geometry>
+      </collision>
+      <inertial>
+        <origin rpy="0 0 0" xyz="0.0138160000 0.0000000000  0.0000000000"/>
+        <mass value="0.016246" />
+        <inertia ixx="0.0000047310" iyy="0.0000015506" izz="0.0000037467" ixy="0.0000004560" ixz="0.0000000000" iyz="0.0000000000" />
+      </inertial>
+    </link>
+  </xacro:macro>
+  <!--///////////////////////////////////////////////////////////////////////////////////////////////////////////////////////////////// -->
   <!-- leddar vu8 8-segment sensor -->
   <xacro:macro name="lidar_leddar_vu8_macro" params="namespace parent_link lidar_name lidar_topic min_angle max_angle min_range max_range *origin">
@@ -770,5 +1015,5 @@
     <xacro:stereo_camera_macro
       namespace="${namespace}"
-      camera_name="vi_sensor"
+      camera_name="${namespace}/vi_sensor"
       parent_link="${parent_link}"
       frame_rate="${frame_rate}"
@@ -875,5 +1120,5 @@
       </visual>
       <inertial>
-        <mass value="0.13" />
+        <mass value="0.001" />
         <origin xyz="0 0 0" rpy="0 0 0" />
         <inertia ixx="1e-6" ixy="0" ixz="0" iyy="1e-6" iyz="0" izz="1e-6" />

File: rotors_description/urdf/firefly_large_landing_gear.xacro (robot description, xacro)
@@ -128,13 +128,13 @@
   <link name="${namespace}_left_leg">
     <visual>
-      <origin xyz="${arm_length*0.013} ${arm_length*0.013} -0.17" rpy="0 0 0" />
-      <geometry>
-        <cylinder length="0.3" radius="0.005"/>
-      </geometry>
-    </visual>
-    <collision>
-      <origin xyz="${arm_length*0.013} ${arm_length*0.013} -0.17" rpy="0 0 0" />
-      <geometry>
-        <cylinder length="0.3" radius="0.005"/>
+      <origin xyz="${arm_length*0.013} ${arm_length*0.013} -0.21" rpy="0 0 0" />
+      <geometry>
+        <cylinder length="0.4" radius="0.005"/>
+      </geometry>
+    </visual>
+    <collision>
+      <origin xyz="${arm_length*0.013} ${arm_length*0.013} -0.21" rpy="0 0 0" />
+      <geometry>
+        <cylinder length="0.4" radius="0.005"/>
       </geometry>
     </collision>
@@ -172,13 +172,13 @@
   <link name="${namespace}_back_left_leg">
     <visual>
-      <origin xyz="-${cos30*arm_length*0.013} ${sin30*arm_length*0.013} -0.17" rpy="0 0 0" />
-      <geometry>
-        <cylinder length="0.3" radius="0.005"/>
-      </geometry>
-    </visual>
-    <collision>
-      <origin xyz="-${cos30*arm_length*0.013} ${sin30*arm_length*0.013} -0.17" rpy="0 0 0" />
-      <geometry>
-        <cylinder length="0.3" radius="0.005"/>
+      <origin xyz="-${cos30*arm_length*0.013} ${sin30*arm_length*0.013} -0.21" rpy="0 0 0" />
+      <geometry>
+        <cylinder length="0.4" radius="0.005"/>
+      </geometry>
+    </visual>
+    <collision>
+      <origin xyz="-${cos30*arm_length*0.013} ${sin30*arm_length*0.013} -0.21" rpy="0 0 0" />
+      <geometry>
+        <cylinder length="0.4" radius="0.005"/>
       </geometry>
     </collision>
@@ -216,13 +216,13 @@
   <link name="${namespace}_back_right_leg">
     <visual>
-      <origin xyz="-${cos30*arm_length*0.013} -${sin30*arm_length*0.013} -0.17" rpy="0 0 0" />
-      <geometry>
-        <cylinder length="0.3" radius="0.005"/>
-      </geometry>
-    </visual>
-    <collision>
-      <origin xyz="-${cos30*arm_length*0.013} -${sin30*arm_length*0.013} -0.17" rpy="0 0 0" />
-      <geometry>
-        <cylinder length="0.3" radius="0.005"/>
+      <origin xyz="-${cos30*arm_length*0.013} -${sin30*arm_length*0.013} -0.21" rpy="0 0 0" />
+      <geometry>
+        <cylinder length="0.4" radius="0.005"/>
+      </geometry>
+    </visual>
+    <collision>
+      <origin xyz="-${cos30*arm_length*0.013} -${sin30*arm_length*0.013} -0.21" rpy="0 0 0" />
+      <geometry>
+        <cylinder length="0.4" radius="0.005"/>
       </geometry>
     </collision>
@@ -261,13 +261,13 @@
   <link name="${namespace}_right_leg">
     <visual>
-      <origin xyz="${arm_length*0.013} -${arm_length*0.013} -0.17" rpy="0 0 0" />
-      <geometry>
-        <cylinder length="0.3" radius="0.005"/>
-      </geometry>
-    </visual>
-    <collision>
-      <origin xyz="${arm_length*0.013} -${arm_length*0.013} -0.17" rpy="0 0 0" />
-      <geometry>
-        <cylinder length="0.3" radius="0.005"/>
+      <origin xyz="${arm_length*0.013} -${arm_length*0.013} -0.21" rpy="0 0 0" />
+      <geometry>
+        <cylinder length="0.4" radius="0.005"/>
+      </geometry>
+    </visual>
+    <collision>
+      <origin xyz="${arm_length*0.013} -${arm_length*0.013} -0.21" rpy="0 0 0" />
+      <geometry>
+        <cylinder length="0.4" radius="0.005"/>
       </geometry>
     </collision>

Commit message: some tuning for manipulator

File: rotors_description/urdf/component_snippets.xacro (robot description, xacro)
@@ -369,5 +369,5 @@
       <inertial>
         <origin rpy="0 0 0" xyz="0.0138160000 0.0000000000 0.0000000000"/>
-          <mass value="0.016246" />
+          <mass value="0.0016246" />
         <inertia ixx="0.0000047310" iyy="0.0000015506" izz="0.0000037467" ixy="-0.0000004560" ixz="0.0000000000" iyz="0.0000000000" />
       </inertial>
@@ -404,5 +404,5 @@
       <inertial>
         <origin rpy="0 0 0" xyz="0.0138160000 0.0000000000  0.0000000000"/>
-        <mass value="0.016246" />
+        <mass value="0.0016246" />
         <inertia ixx="0.0000047310" iyy="0.0000015506" izz="0.0000037467" ixy="0.0000004560" ixz="0.0000000000" iyz="0.0000000000" />
       </inertial>

File: rotors_description/urdf/firefly_large_landing_gear.xacro (robot description, xacro)
@@ -185,5 +185,5 @@
     <inertial>
       <origin rpy="0.0 0.0 0.0" xyz="0.0 0.0 0.0"/>
-      <mass value="0.0230" />
+      <mass value="0.0145" />
       <inertia ixx="0.0021150000" iyy="0.0006921000" izz="0.0025240000" ixy="-0.0000163500" ixz="0.0000006998" iyz="0.0000464200" />
     </inertial>
@@ -229,5 +229,5 @@
     <inertial>
       <origin rpy="0.0 0.0 0.0" xyz="0.0 0.0 0.0"/>
-      <mass value="0.0230" />
+      <mass value="0.0120" />
       <inertia ixx="0.0021150000" iyy="0.0006921000" izz="0.0025240000" ixy="-0.0000163500" ixz="0.0000006998" iyz="0.0000464200" />
     </inertial>
